File: hardware/KiCad/jjy_sim_r3.kicad_sch (KiCad schematic)
At the start: 60 parts, among them P1 USB_C_Plug_USB2.0, Q1 HN1C01FU-GR, SW1 RESET, SW2 CONFIG, SW3 BAND, U1 AM1025EA, U2 ESP32-C3-WROOM-02, U3 RT9193-33GB, U4 UG-2864HL, U5 CH340K

Commit message: Update project for KiCad 10.0 and add local libraries
- Updated KiCad project files for KiCad 10.0
- Moved the BAND-SW position
- Added project-local KiCad libraries
- Included custom libraries that were previously not committed
Parts:
- JP1, JP2: footprint MY_LIB:Jumper-2_TH_3.81mm -> JJY-SIM-R3:Jumper-2_TH_3.81mm
- P1: footprint MY_LIB:5077CR-16SMC2-BK-TR -> JJY-SIM-R3:5077CR-16SMC2-BK-TR_Ext
- Q1: footprint MY_LIB:2-2J1A -> JJY-SIM-R3:2-2J1A
- SW1: renamed from SW3; footprint MY_LIB:MSK-12C02 -> JJY-SIM-R3:MSK-12C02
- SW2: renamed from SW1; footprint MY_LIB:SKRPACE010 -> JJY-SIM-R3:SKRPACE010; symbol MY_LIB:SW_PUSH2 -> JJY-SIM-R3_Library:SW_PUSH2
- SW3: renamed from SW2; footprint MY_LIB:SKRPACE010 -> JJY-SIM-R3:SKRPACE010; symbol MY_LIB:SW_PUSH2 -> JJY-SIM-R3_Library:SW_PUSH2
- TP1, TP2, TP3: symbol MY_LIB:TP -> Connector:TestPoint
- U1: footprint MY_LIB:eSOP-8_3.9x5.05mm_EP_3.1x2.2mm_P1.27mm -> JJY-SIM-R3:eSOP-8_3.9x5.05mm_EP_3.1x2.2mm_P1.27mm
- U2: renamed from U5; footprint Package_SO:SSOP-10-1EP_3.9x4.9mm_P1mm_EP2.1x3.3mm -> JJY-SIM-R3:SSOP-10-1EP_3.9x4.9mm_P1mm_EP2.1x3.3mm; KiLib_Generator (none) -> package/gullwing
- U3: renamed from U2; footprint RF_Module:ESP32-C3-WROOM-02 -> JJY-SIM-R3:ESP32-C3-WROOM-02,ESP8684-WROOM-2C; symbol Espressif:ESP32-C3-WROOM-02 -> JJY-SIM-R3_Library:ESP32-C3-WROOM-02
- U4: renamed from U3; symbol MY_LIB:RT9193-33GB -> JJY-SIM-R3_Library:RT9193-33GB
- U5: renamed from U4; footprint MY_LIB:UG-2864-FPC -> JJY-SIM-R3:UG-2864-FPC (Reverse); symbol MY_LIB:UG-286HL -> JJY-SIM-R3_Library:UG-2864
- renumbered C9 to C10, C10 to C11, C11 to C12, C6 to C13, C17 to C14, C16 to C15, C15 to C16, C14 to C17, C13 to C18, C12 to C19, C3 to C2, C2 to C3, C19 to C6, C18 to C8, C8 to C9, D2 to D1, D3 to D2, D4 to D3, D7 to D4, R7 to R1, R12 to R10, R19 to R11, R20 to R12, R21 to R13, R22 to R14, R17 to R16, R16 to R17, R13 to R19, R5 to R2, R14 to R20, R2 to R3, R6 to R5, R8 to R6, R9 to R7, R10 to R8, R11 to R9
Connections:
- net RF_A: now also R2.1, R3.1; no longer C4.2, C5.2
- net RF_B: now also C3.2, SW1.2 (B); no longer R2.1, R3.1
- net at C4.1, C5.1: now also U1.5 (OUT_B); no longer C3.2, SW1.3 (C)
- net at R2.2, R3.2: now also U1.7 (OUT_A); no longer U1.5 (OUT_B)
- net at SW1.1 (A): now also C3.1, C4.2, C5.2
Other:
- moved on the sheet: C13, C3, C4, C5, D1, D2, D3, R2, R3, R7, R8, R9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
